Commit message: visualized the point cloud

File: urdf/sensorRig1_description.urdf (robot description, URDF)
Before this commit: robot sensorRig1, 2 links, 1 joints
Links:
- removed link guidance
- added link camera
Joints:
- removed joint base_to_guidance
- added joint base_to_camera: type fixed, parent base_link, child camera, origin xyz=0 0 0.06 rpy=1.5707963268 3.14159265359 1.5707963268
